Commit message: fix xacro origin bug

File: mgs1600gy_description/urdf/mgs1600gy.urdf.xacro (robot description, xacro)
@@ -8,7 +8,7 @@
       prefix=""
       parent="base_link">
-    <origin
-        xyz="0 0 0"
-        rpy="0 0 0" />
+      <origin
+          xyz="0.015 0 0"
+          rpy="0 0 0" />
   </xacro:mgs1600gy>
 </robot>

File: mgs1600gy_description/urdf/mgs1600gy.xacro (robot description, xacro)
@@ -12,9 +12,7 @@
         name="${prefix}mgs1600gy_joint"
         type="fixed">
-      <origin
-          xyz="0.015 0 0"
-          rpy="0 0 0" />
       <parent link="${parent}" />
       <child link="${prefix}mgs1600gy_link" />
+      <xacro:insert_block name="origin" />
     </joint>
     <link name="${prefix}mgs1600gy_link">

Commit message: add gazebo check for description file

File: mgs1600gy_description/urdf/mgs1600gy.urdf.xacro (robot description, xacro)
@@ -7,8 +7,9 @@
   <xacro:mgs1600gy
       prefix=""
-      parent="base_link">
-      <origin
-          xyz="0.015 0 0"
-          rpy="0 0 0" />
+      parent="base_link"
+      is_gazebo="False">
+    <origin
+        xyz="0.015 0 0"
+        rpy="0 0 0" />
   </xacro:mgs1600gy>
 </robot>

File: mgs1600gy_description/urdf/mgs1600gy.xacro (robot description, xacro)
@@ -8,5 +8,5 @@
   <xacro:macro
       name="mgs1600gy"
-      params="parent prefix *origin">
+      params="parent prefix is_gazebo *origin">
     <!-- Links -->
     <link name="${prefix}mgs1600gy_link">
@@ -41,9 +41,4 @@
       </collision>
     </link>
-    <link name="${prefix}mgs1600gy_sensor_link">
-      <inertial>
-        <mass value="0.0" />
-      </inertial>
-    </link>
     <!-- Joints -->
     <joint
@@ -54,47 +49,64 @@
       <xacro:insert_block name="origin" />
     </joint>
-    <joint
-        name="${prefix}mgs1600gy_sensor_joint"
-        type="fixed">
-      <parent link="${prefix}mgs1600gy_link" />
-      <child link="${prefix}mgs1600gy_sensor_link" />
-      <origin
-          xyz="0 0 ${220.0 * const.SCALE_MM}"
-          rpy="0 ${const.TO_RADIAN * 90} 0" />
-    </joint>
     <!-- Gazebo -->
-    <gazebo reference="${prefix}mgs1600gy_sensor_link">
-      <sensor
-          type="camera"
-          name="${prefix}mgs1600gy">
-        <update_rate>10.0</update_rate>
-        <always_on>true</always_on>
-        <visualize>true</visualize>
-        <camera name="head">
-          <image>
-            <width>160</width>
-            <height>1</height>
-            <format>R8G8B8</format>
-          </image>
-          <clip>
-            <near>0.23</near>
-            <far>300</far>
-          </clip>
-          <noise>
-            <type>gaussian</type>
-            <mean>0.0</mean>
-            <stddev>0.001</stddev>
-          </noise>
-        </camera>
-        <!-- success -->
-        <plugin
-            name="camera_controller"
-            filename="libgazebo_ros_camera.so">
-          <alwaysOn>true</alwaysOn>
-          <camera_name>${prefix}mgs1600gy</camera_name>
-          <frame_name>${prefix}mgs1600gy_link</frame_name>
-        </plugin>
-      </sensor>
-    </gazebo>
+    <xacro:if value="${is_gazebo}">
+      <link name="${prefix}mgs1600gy_sensor_link">
+        <inertial>
+          <origin
+              xyz="0 0 0"
+              rpy="0 0 0" />
+          <mass value="0.0" />
+          <inertia
+              ixx="0"
+              ixy="0"
+              ixz="0"
+              iyy="0"
+              iyz="0"
+              izz="0" />
+        </inertial>
+      </link>
+      <joint
+          name="${prefix}mgs1600gy_sensor_joint"
+          type="fixed">
+        <parent link="${prefix}mgs1600gy_link" />
+        <child link="${prefix}mgs1600gy_sensor_link" />
+        <origin
+            xyz="0 0 ${220.0 * const.SCALE_MM}"
+            rpy="0 ${const.TO_RADIAN * 90} 0" />
+      </joint>
+      <gazebo reference="${prefix}mgs1600gy_sensor_link">
+        <sensor
+            type="camera"
+            name="${prefix}mgs1600gy">
+          <update_rate>10.0</update_rate>
+          <always_on>true</always_on>
+          <visualize>true</visualize>
+          <camera name="head">
+            <image>
+              <width>160</width>
+              <height>1</height>
+              <format>R8G8B8</format>
+            </image>
+            <clip>
+              <near>0.23</near>
+              <far>300</far>
+            </clip>
+            <noise>
+              <type>gaussian</type>
+              <mean>0.0</mean>
+              <stddev>0.001</stddev>
+            </noise>
+          </camera>
+          <!-- success -->
+          <plugin
+              name="camera_controller"
+              filename="libgazebo_ros_camera.so">
+            <alwaysOn>true</alwaysOn>
+            <camera_name>${prefix}mgs1600gy</camera_name>
+            <frame_name>${prefix}mgs1600gy_link</frame_name>
+          </plugin>
+        </sensor>
+      </gazebo>
+    </xacro:if>
   </xacro:macro>
 </robot>

Commit message: add flip function to gazebo sensor

File: mgs1600gy_description/urdf/mgs1600gy.urdf.xacro (robot description, xacro)
@@ -7,6 +7,5 @@
   <xacro:mgs1600gy
       prefix=""
-      parent="base_link"
-      is_gazebo="False">
+      parent="base_link" >
     <origin
         xyz="0.015 0 0"

File: mgs1600gy_description/urdf/mgs1600gy.xacro (robot description, xacro)
@@ -8,5 +8,5 @@
   <xacro:macro
       name="mgs1600gy"
-      params="parent prefix is_gazebo *origin">
+      params="parent prefix is_gazebo:=False flip:=False *origin">
     <!-- Links -->
     <link name="${prefix}mgs1600gy_link">
@@ -71,7 +71,14 @@
         <parent link="${prefix}mgs1600gy_link" />
         <child link="${prefix}mgs1600gy_sensor_link" />
-        <origin
-            xyz="0 0 ${220.0 * const.SCALE_MM}"
-            rpy="0 ${const.TO_RADIAN * 90} 0" />
+        <xacro:if value="${flip}">
+          <origin
+              xyz="0 0 ${180.0 * const.SCALE_MM}"
+              rpy="0 ${const.TO_RADIAN * 90.0} ${180.0 * const.TO_RADIAN}" />
+        </xacro:if>
+        <xacro:unless value="${flip}">
+          <origin
+              xyz="0 0 ${180.0 * const.SCALE_MM}"
+              rpy="0 ${const.TO_RADIAN * 90.0} 0" />
+        </xacro:unless>
       </joint>
       <gazebo reference="${prefix}mgs1600gy_sensor_link">
@@ -86,8 +93,8 @@
               <width>160</width>
               <height>1</height>
-              <format>R8G8B8</format>
+              <format>L8</format>
             </image>
             <clip>
-              <near>0.23</near>
+              <near>0.19</near>
               <far>300</far>
             </clip>

Commit message: add sensor link

File: mgs1600gy_description/urdf/mgs1600gy.urdf.xacro (robot description, xacro)
@@ -4,8 +4,14 @@
     name="mgs1600gy">
   <xacro:include filename="$(find mgs1600gy_description)/urdf/mgs1600gy.xacro" />
+  <!-- arguments -->
+  <xacro:arg
+      name="use_nominal_extrinsics"
+      default="False" />
   <link name="base_link" />
   <xacro:mgs1600gy
       prefix=""
-      parent="base_link" >
+      parent="base_link"
+      use_nominal_extrinsics="$(arg use_nominal_extrinsics)"
+      >
     <origin
         xyz="0.015 0 0"

File: mgs1600gy_description/urdf/mgs1600gy.xacro (robot description, xacro)
@@ -5,5 +5,5 @@
   <xacro:macro
       name="mgs1600gy"
-      params="parent prefix is_gazebo:=False flip:=False *origin">
+      params="parent prefix is_gazebo:=False flip:=False  use_nominal_extrinsics:=False *origin">
     <!-- Links -->
     <link name="${prefix}mgs1600gy_link">
@@ -38,4 +38,30 @@
       </collision>
     </link>
+    <xacro:if value="${use_nominal_extrinsics}">
+      <!-- Magnet sensor link -->
+      <link name="${prefix}mgs1600gy_magnet_link" />
+      <joint
+          name="${prefix}mgs1600gy_magnet_joint"
+          type="fixed">
+        <parent link="${prefix}mgs1600gy_link" />
+        <child link="${prefix}mgs1600gy_magnet_link" />
+        <!-- TODO(m12watanabe1a) fix origin -->
+        <origin
+            xyz="0 0 0"
+            rpy="0 0 0" />
+      </joint>
+      <!-- Gyro sensor link -->
+      <link name="${prefix}mgs1600gy_gyro_link" />
+      <joint
+          name="${prefix}mgs1600gy_gyro_joint"
+          type="fixed">
+        <parent link="${prefix}mgs1600gy_link" />
+        <child link="${prefix}mgs1600gy_gyro_link" />
+        <!-- TODO(m12watanabe1a) fix origin -->
+        <origin
+            xyz="0 0 0"
+            rpy="0 0 0" />
+      </joint>
+    </xacro:if>
     <!-- Joints -->
     <joint

Commit message: add calibration code

File: mgs1600gy_description/urdf/mgs1600gy.urdf.xacro (robot description, xacro)
@@ -12,8 +12,7 @@
       prefix=""
       parent="base_link"
-      use_nominal_extrinsics="$(arg use_nominal_extrinsics)"
-      >
+      use_nominal_extrinsics="$(arg use_nominal_extrinsics)">
     <origin
-        xyz="0.015 0 0"
+        xyz="0.5 0 1"
         rpy="0 0 0" />
   </xacro:mgs1600gy>

File: mgs1600gy_description/urdf/mgs1600gy.xacro (robot description, xacro)
@@ -39,4 +39,23 @@
     </link>
     <xacro:if value="${use_nominal_extrinsics}">
+      <!-- Gyro sensor link -->
+      <!-- Joints -->
+      <joint
+          name="${prefix}mgs1600gy_joint"
+          type="floating">
+        <parent link="${parent}" />
+        <child link="${prefix}mgs1600gy_gyro_link" />
+        <xacro:insert_block name="origin" />
+      </joint>
+      <link name="${prefix}mgs1600gy_gyro_link" />
+      <joint
+          name="${prefix}mgs1600gy_gyro_joint"
+          type="fixed">
+        <parent link="${prefix}mgs1600gy_gyro_link" />
+        <child link="${prefix}mgs1600gy_link" />
+        <origin
+            xyz="0 0 -12.5E-03"
+            rpy="0 0 0" />
+      </joint>
       <!-- Magnet sensor link -->
       <link name="${prefix}mgs1600gy_magnet_link" />
@@ -50,24 +69,15 @@
             rpy="0 0 0" />
       </joint>
-      <!-- Gyro sensor link -->
-      <link name="${prefix}mgs1600gy_gyro_link" />
+    </xacro:if>
+    <xacro:unless value="${use_nominal_extrinsics}">
+      <!-- Joints -->
       <joint
-          name="${prefix}mgs1600gy_gyro_joint"
+          name="${prefix}mgs1600gy_joint"
           type="fixed">
-        <parent link="${prefix}mgs1600gy_link" />
-        <child link="${prefix}mgs1600gy_gyro_link" />
-        <origin
-            xyz="0 0 12.5E-03"
-            rpy="0 0 0" />
+        <parent link="${parent}" />
+        <child link="${prefix}mgs1600gy_link" />
+        <xacro:insert_block name="origin" />
       </joint>
-    </xacro:if>
-    <!-- Joints -->
-    <joint
-        name="${prefix}mgs1600gy_joint"
-        type="fixed">
-      <parent link="${parent}" />
-      <child link="${prefix}mgs1600gy_link" />
-      <xacro:insert_block name="origin" />
-    </joint>
+    </xacro:unless>
     <!-- Gazebo -->
     <xacro:if value="${is_gazebo}">
