Commit message: kurimoto adds inertia

File: mgs1600gy_description/urdf/mgs1600gy.xacro (robot description, xacro)
@@ -19,6 +19,14 @@
       <visual>
         <origin
-            xyz="0 0 0"
+            xyz="-1.718E-03 -1.635E-03 13.993E-03"
             rpy="0 0 0" />
+        <mass value="3.75E-02" />
+        <inertia
+            ixx="8.56E-05"
+            ixy="-1.25E-07"
+            ixz="4.65E-07"
+            iyy="7.79E-06"
+            iyz="5.94E-07"
+            izz="8.56E-05" />
         <geometry>
           <mesh filename="package://mgs1600gy_description/meshes/body.dae" />

Commit message: fix inertial bug tag

File: mgs1600gy_description/urdf/mgs1600gy.xacro (robot description, xacro)
@@ -17,5 +17,5 @@
     </joint>
     <link name="${prefix}mgs1600gy_link">
-      <visual>
+      <inertial>
         <origin
             xyz="-1.718E-03 -1.635E-03 13.993E-03"
@@ -29,4 +29,9 @@
             iyz="5.94E-07"
             izz="8.56E-05" />
+      </inertial>
+      <visual>
+        <origin
+            xyz="0 0 0"
+            rpy="0 0 0" />
         <geometry>
           <mesh filename="package://mgs1600gy_description/meshes/body.dae" />

Commit message: add gazebo sensor plugin

File: mgs1600gy_description/urdf/mgs1600gy.xacro (robot description, xacro)
@@ -9,11 +9,5 @@
       name="mgs1600gy"
       params="parent prefix *origin">
-    <joint
-        name="${prefix}mgs1600gy_joint"
-        type="fixed">
-      <parent link="${parent}" />
-      <child link="${prefix}mgs1600gy_link" />
-      <xacro:insert_block name="origin" />
-    </joint>
+    <!-- Links -->
     <link name="${prefix}mgs1600gy_link">
       <inertial>
@@ -47,4 +41,60 @@
       </collision>
     </link>
+    <link name="${prefix}mgs1600gy_sensor_link">
+      <inertial>
+        <mass value="0.0" />
+      </inertial>
+    </link>
+    <!-- Joints -->
+    <joint
+        name="${prefix}mgs1600gy_joint"
+        type="fixed">
+      <parent link="${parent}" />
+      <child link="${prefix}mgs1600gy_link" />
+      <xacro:insert_block name="origin" />
+    </joint>
+    <joint
+        name="${prefix}mgs1600gy_sensor_joint"
+        type="fixed">
+      <parent link="${prefix}mgs1600gy_link" />
+      <child link="${prefix}mgs1600gy_sensor_link" />
+      <origin
+          xyz="0 0 ${220.0 * const.SCALE_MM}"
+          rpy="0 ${const.TO_RADIAN * 90} 0" />
+    </joint>
+    <!-- Gazebo -->
+    <gazebo reference="${prefix}mgs1600gy_sensor_link">
+      <sensor
+          type="camera"
+          name="${prefix}mgs1600gy">
+        <update_rate>10.0</update_rate>
+        <always_on>true</always_on>
+        <visualize>true</visualize>
+        <camera name="head">
+          <image>
+            <width>160</width>
+            <height>1</height>
+            <format>R8G8B8</format>
+          </image>
+          <clip>
+            <near>0.23</near>
+            <far>300</far>
+          </clip>
+          <noise>
+            <type>gaussian</type>
+            <mean>0.0</mean>
+            <stddev>0.001</stddev>
+          </noise>
+        </camera>
+        <!-- success -->
+        <plugin
+            name="camera_controller"
+            filename="libgazebo_ros_camera.so">
+          <alwaysOn>true</alwaysOn>
+          <camera_name>${prefix}mgs1600gy</camera_name>
+          <frame_name>${prefix}mgs1600gy_link</frame_name>
+        </plugin>
+      </sensor>
+    </gazebo>
   </xacro:macro>
 </robot>

Commit message: add gazebo plugin

File: mgs1600gy_description/urdf/mgs1600gy.xacro (robot description, xacro)
@@ -51,44 +51,19 @@
     <!-- Gazebo -->
     <xacro:if value="${is_gazebo}">
-      <link name="${prefix}mgs1600gy_sensor_link">
-        <inertial>
-          <origin
-              xyz="0 0 0"
-              rpy="0 0 0" />
-          <mass value="0.0" />
-          <inertia
-              ixx="0"
-              ixy="0"
-              ixz="0"
-              iyy="0"
-              iyz="0"
-              izz="0" />
-        </inertial>
-      </link>
-      <joint
-          name="${prefix}mgs1600gy_sensor_joint"
-          type="fixed">
-        <parent link="${prefix}mgs1600gy_link" />
-        <child link="${prefix}mgs1600gy_sensor_link" />
-        <xacro:if value="${flip}">
-          <origin
-              xyz="0 0 ${180.0 * const.SCALE_MM}"
-              rpy="0 ${const.TO_RADIAN * 90.0} ${180.0 * const.TO_RADIAN}" />
-        </xacro:if>
-        <xacro:unless value="${flip}">
-          <origin
-              xyz="0 0 ${180.0 * const.SCALE_MM}"
-              rpy="0 ${const.TO_RADIAN * 90.0} 0" />
-        </xacro:unless>
-      </joint>
-      <!--
-      <gazebo reference="${prefix}mgs1600gy_sensor_link">
+      <gazebo reference="${prefix}mgs1600gy_link">
         <sensor
-            type="camera"
+            type="segmentation"
             name="${prefix}mgs1600gy">
           <update_rate>10.0</update_rate>
           <always_on>true</always_on>
           <visualize>true</visualize>
-          <camera name="head">
+          <topic>/mgs/${prefix}</topic>
+          <xacro:if value="${flip}">
+            <pose>0 0 0.18 0 ${90.0 * const.TO_RADIAN} ${180.0 * const.TO_RADIAN}</pose>
+          </xacro:if>
+          <xacro:unless value="${flip}">
+            <pose>0 0 0.18 0 ${90.0 * const.TO_RADIAN} 0</pose>
+          </xacro:unless>
+          <camera>
             <image>
               <width>160</width>
@@ -100,20 +75,7 @@
               <far>300</far>
             </clip>
-            <noise>
-              <type>gaussian</type>
-              <mean>0.0</mean>
-              <stddev>0.001</stddev>
-            </noise>
           </camera>
-      <plugin
-          name="camera_controller"
-          filename="libgazebo_ros_camera.so">
-        <alwaysOn>true</alwaysOn>
-        <camera_name>${prefix}mgs1600gy</camera_name>
-        <frame_name>${prefix}mgs1600gy_link</frame_name>
-      </plugin>
-      </sensor>
+        </sensor>
       </gazebo>
-      -->
     </xacro:if>
   </xacro:macro>

Commit message: Update mgs1600gy.xacro

File: mgs1600gy_description/urdf/mgs1600gy.xacro (robot description, xacro)
@@ -3,7 +3,4 @@
     xmlns:xacro="http://ros.org/wiki/xacro"
     name="mgs1600gy">
-  <xacro:property
-      name="MGS1600GY_BODY_LINK"
-      value="mgs1600gy_description/meshes/body.stl" />
   <xacro:macro
       name="mgs1600gy"

Commit message: fix urdf

File: mgs1600gy_description/urdf/mgs1600gy.xacro (robot description, xacro)
@@ -9,5 +9,5 @@
   <xacro:macro
       name="mgs1600gy"
-      params="parent prefix is_gazebo:=False flip:=False  use_nominal_extrinsics:=False *origin">
+      params="parent prefix is_gazebo:=False flip:=False use_nominal_extrinsics:=False *origin">
     <!-- Links -->
     <link name="${prefix}mgs1600gy_link">
@@ -43,23 +43,4 @@
     </link>
     <xacro:if value="${use_nominal_extrinsics}">
-      <!-- Gyro sensor link -->
-      <!-- Joints -->
-      <joint
-          name="${prefix}mgs1600gy_joint"
-          type="floating">
-        <parent link="${parent}" />
-        <child link="${prefix}mgs1600gy_gyro_link" />
-        <xacro:insert_block name="origin" />
-      </joint>
-      <link name="${prefix}mgs1600gy_gyro_link" />
-      <joint
-          name="${prefix}mgs1600gy_gyro_joint"
-          type="fixed">
-        <parent link="${prefix}mgs1600gy_gyro_link" />
-        <child link="${prefix}mgs1600gy_link" />
-        <origin
-            xyz="0 0 -12.5E-03"
-            rpy="0 0 0" />
-      </joint>
       <!-- Magnet sensor link -->
       <link name="${prefix}mgs1600gy_magnet_link" />
@@ -74,14 +55,12 @@
       </joint>
     </xacro:if>
-    <xacro:unless value="${use_nominal_extrinsics}">
-      <!-- Joints -->
-      <joint
-          name="${prefix}mgs1600gy_joint"
-          type="fixed">
-        <parent link="${parent}" />
-        <child link="${prefix}mgs1600gy_link" />
-        <xacro:insert_block name="origin" />
-      </joint>
-    </xacro:unless>
+    <!-- Joints -->
+    <joint
+        name="${prefix}mgs1600gy_joint"
+        type="fixed">
+      <parent link="${parent}" />
+      <child link="${prefix}mgs1600gy_link" />
+      <xacro:insert_block name="origin" />
+    </joint>
     <!-- Gazebo -->
     <xacro:if value="${is_gazebo}">
